File: 32u4/GMcounter.sch (KiCad schematic (older format))
At the start: 44 parts, among them J1 Conn_02x05_Counter_Clockwise, P1 CONN_01X01, P2 CONN_01X01, P3 CONN_01X01, P4 USB_A, P5 CONN_01X03, P7 CONN_01X03, Q1 MMBT3904, Q2 STL128DN, Q3 MMBT3904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

Commit message: first version to printer
Parts:
- C1, C2, C3, C4, C6: symbol GMcounter-rescue:CP -> GMcounter-rescue:CP-GMcounter-rescue
- C5, C7, C8, C9: symbol GMcounter-rescue:C -> GMcounter-rescue:C-GMcounter-rescue
- D1, D2, D5: symbol GMcounter-rescue:D -> GMcounter-rescue:D-GMcounter-rescue
- D3, D4: symbol GMcounter-rescue:LED -> GMcounter-rescue:LED-GMcounter-rescue
- L1: footprint Inductors:SELF-WE-PD-XXL -> MyKiCadLibs:SRR1208; symbol GMcounter-rescue:L_Small -> GMcounter-rescue:L_Small-GMcounter-rescue
- P1, P2, P3: symbol GMcounter-rescue:CONN_01X01 -> GMcounter-rescue:CONN_01X01-GMcounter-rescue
- P4: symbol GMcounter-rescue:USB_A -> GMcounter-rescue:USB_A-GMcounter-rescue
- P5, P7: symbol GMcounter-rescue:CONN_01X03 -> GMcounter-rescue:CONN_01X03-GMcounter-rescue
- Q1, Q3: symbol GMcounter-rescue:MMBT3904 -> GMcounter-rescue:MMBT3904-GMcounter-rescue
- Q2: symbol GMcounter-rescue:BD249C -> GMcounter-rescue:BD249C-GMcounter-rescue
- Q4: symbol GMcounter-rescue:CSTLA_T -> GMcounter-rescue:CSTLA_T-GMcounter-rescue
- R1, R10, R11, R12, R13, R14, R2, R3, R4, R5, R6, R7, R8, R9: symbol GMcounter-rescue:R -> GMcounter-rescue:R-GMcounter-rescue
- RV1: symbol GMcounter-rescue:POT -> GMcounter-rescue:POT-GMcounter-rescue
- U1: symbol GMcounter-rescue:TLC555CP -> GMcounter-rescue:TLC555CP-GMcounter-rescue
- U2: symbol GMcounter-rescue:ATmega32U4 -> GMcounter-rescue:ATmega32U4-GMcounter-rescue
- U3: symbol GMcounter-rescue:AP1117D33 -> GMcounter-rescue:AP1117D33-GMcounter-rescue
Changed lines of the file:
@@
 $EndDescr
 $Comp
-L GMcounter-rescue:TLC555CP U1
+L GMcounter-rescue:TLC555CP-GMcounter-rescue U1
 U 1 1 5BE0E0C5
 P 1900 2700
@@
 $EndComp
 $Comp
-L GMcounter-rescue:GND #PWR01
+L GMcounter-rescue:GND-GMcounter-rescue #PWR01
 U 1 1 5BE0E4DE
 P 2500 4100
@@
 Connection ~ 2500 3150
 $Comp
-L GMcounter-rescue:R R1
+L GMcounter-rescue:R-GMcounter-rescue R1
 U 1 1 5BE0E558
 P 950 2750
@@
 Connection ~ 1900 3150
 $Comp
-L GMcounter-rescue:R R3
+L GMcounter-rescue:R-GMcounter-rescue R3
 U 1 1 5BE0E66E
 P 3100 2500
@@
 $EndComp
 $Comp
-L GMcounter-rescue:R R2
+L GMcounter-rescue:R-GMcounter-rescue R2
 U 1 1 5BE0E6B1
 P 2850 2850
@@
 $EndComp
 $Comp
-L GMcounter-rescue:D D1
+L GMcounter-rescue:D-GMcounter-rescue D1
 U 1 1 5BE0E6DC
 P 2850 3250
@@
 	2850 3100 2850 3000
 $Comp
-L GMcounter-rescue:CP C1
+L GMcounter-rescue:CP-GMcounter-rescue C1
 U 1 1 5BE0E83A
 P 2850 3750
@@
 Connection ~ 3350 2500
 $Comp
-L GMcounter-rescue:L_Small L1
+L GMcounter-rescue:L_Small-GMcounter-rescue L1
 U 1 1 5BE0ED37
 P 3900 1900
 F 0 "L1" H 3750 1950 50  0000 L CNN
 F 1 "10mH" H 3550 1850 50  0000 L CNN
-F 2 "Inductors:SELF-WE-PD-XXL" H 3900 1900 50  0001 C CNN
+F 2 "MyKiCadLibs:SRR1208" H 3900 1900 50  0001 C CNN
 F 3 "" H 3900 1900 50  0000 C CNN
 	1    3900 1900
@@
 $EndComp
 $Comp
-L GMcounter-rescue:D D2
+L GMcounter-rescue:D-GMcounter-rescue D2
 U 1 1 5BE0ED74
 P 4250 2150
@@
 $EndComp
 $Comp
-L GMcounter-rescue:CP C2
+L GMcounter-rescue:CP-GMcounter-rescue C2
 U 1 1 5BE0EDC8
 P 4750 2550
@@
 $EndComp
 $Comp
-L GMcounter-rescue:GND #PWR02
+L GMcounter-rescue:GND-GMcounter-rescue #PWR02
 U 1 1 5BE0EE6A
 P 4750 2900
@@
 Connection ~ 3900 2150
 $Comp
-L GMcounter-rescue:R R6
+L GMcounter-rescue:R-GMcounter-rescue R6
 U 1 1 5BE0EEF9
 P 5100 2150
@@
 	3900 2700 3900 3350
 $Comp
-L GMcounter-rescue:R R4
+L GMcounter-rescue:R-GMcounter-rescue R4
 U 1 1 5BE0F23A
 P 3500 2000
@@
 	3500 3150 3500 2250
 $Comp
-L GMcounter-rescue:+3.3V #PWR03
+L GMcounter-rescue:+3.3V-GMcounter-rescue #PWR03
 U 1 1 5BE0F465
 P 3300 1200
@@
 Connection ~ 3500 1650
 $Comp
-L GMcounter-rescue:R R5
+L GMcounter-rescue:R-GMcounter-rescue R5
 U 1 1 5BE0F516
 P 3900 3650
@@
 Connection ~ 3900 3350
 $Comp
-L GMcounter-rescue:GND #PWR04
+L GMcounter-rescue:GND-GMcounter-rescue #PWR04
 U 1 1 5BE0F743
 P 3500 4800
@@
 	5250 2150 5550 2150
 $Comp
-L GMcounter-rescue:CONN_01X01 P1
+L GMcounter-rescue:CONN_01X01-GMcounter-rescue P1
 U 1 1 5BE0FB6C
 P 5750 2150
@@
 $EndComp
 $Comp
-L GMcounter-rescue:CONN_01X01 P2
+L GMcounter-rescue:CONN_01X01-GMcounter-rescue P2
 U 1 1 5BE0FDC9
 P 750 5100
@@
 $EndComp
 $Comp
-L GMcounter-rescue:CP C3
+L GMcounter-rescue:CP-GMcounter-rescue C3
 U 1 1 5BE0FE37
 P 1200 5600
@@
 $EndComp
 $Comp
-L GMcounter-rescue:R R7
+L GMcounter-rescue:R-GMcounter-rescue R7
 U 1 1 5BE0FEB0
 P 1600 5350
@@
 $EndComp
 $Comp
-L GMcounter-rescue:R R8
+L GMcounter-rescue:R-GMcounter-rescue R8
 U 1 1 5BE0FFA5
 P 1600 5900
@@
 $EndComp
 $Comp
-L GMcounter-rescue:GND #PWR05
+L GMcounter-rescue:GND-GMcounter-rescue #PWR05
 U 1 1 5BE10009
 P 1600 6250
@@
 Connection ~ 1600 6150
 $Comp
-L GMcounter-rescue:R R9
+L GMcounter-rescue:R-GMcounter-rescue R9
 U 1 1 5BE1027E
 P 2250 5100
@@
 $EndComp
 $Comp
-L GMcounter-rescue:+3.3V #PWR06
+L GMcounter-rescue:+3.3V-GMcounter-rescue #PWR06
 U 1 1 5BE102E8
 P 2250 4750
@@
 Connection ~ 1600 5650
 $Comp
-L GMcounter-rescue:CONN_01X01 P3
+L GMcounter-rescue:CONN_01X01-GMcounter-rescue P3
 U 1 1 5BE104B3
 P 2900 5050
@@
 Connection ~ 2250 5350
 $Comp
-L GMcounter-rescue:POT RV1
+L GMcounter-rescue:POT-GMcounter-rescue RV1
 U 1 1 5BE10E85
 P 3900 4150
@@
 Connection ~ 3900 3900
 $Comp
-L GMcounter-rescue:MMBT3904 Q3
+L GMcounter-rescue:MMBT3904-GMcounter-rescue Q3
 U 1 1 5BE1A585
 P 2150 5650
@@
 $EndComp
 $Comp
-L GMcounter-rescue:MMBT3904 Q1
+L GMcounter-rescue:MMBT3904-GMcounter-rescue Q1
 U 1 1 5BE1A698
 P 3600 3350
@@
 $EndComp
 $Comp
-L GMcounter-rescue:BD249C Q2
+L GMcounter-rescue:BD249C-GMcounter-rescue Q2
 U 1 1 5BE1A814
 P 3800 2500
@@
 $EndComp
 $Comp
-L GMcounter-rescue:ATmega32U4 U2
+L GMcounter-rescue:ATmega32U4-GMcounter-rescue U2
 U 1 1 5BE1AC37
 P 8050 2700
@@
 $EndComp
 $Comp
-L GMcounter-rescue:AP1117D33 U3
+L GMcounter-rescue:AP1117D33-GMcounter-rescue U3
 U 1 1 5BE1BC0C
 P 2500 7450
@@
 $EndComp
 $Comp
-L GMcounter-rescue:C C5
+L GMcounter-rescue:C-GMcounter-rescue C5
 U 1 1 5BE1BDB3
 P 2950 7200
@@
 $EndComp
 $Comp
-L GMcounter-rescue:CP C4
+L GMcounter-rescue:CP-GMcounter-rescue C4
 U 1 1 5BE1BE10
 P 3200 7200
@@
 $EndComp
 $Comp
-L GMcounter-rescue:+5V #PWR07
+L GMcounter-rescue:+5V-GMcounter-rescue #PWR07
 U 1 1 5BE1C0A2
 P 3550 7450
@@
 $EndComp
 $Comp
-L GMcounter-rescue:GND #PWR08
+L GMcounter-rescue:GND-GMcounter-rescue #PWR08
 U 1 1 5BE1C105
 P 2500 6500
@@
 $EndComp
 $Comp
-L GMcounter-rescue:C C7
+L GMcounter-rescue:C-GMcounter-rescue C7
 U 1 1 5BE1C1CF
 P 1750 7200
@@
 $EndComp
 $Comp
-L GMcounter-rescue:CP C6
+L GMcounter-rescue:CP-GMcounter-rescue C6
 U 1 1 5BE1C1D5
 P 2000 7200
@@
 	3550 7450 3450 7450
 $Comp
-L GMcounter-rescue:+3.3V #PWR09
+L GMcounter-rescue:+3.3V-GMcounter-rescue #PWR09
 U 1 1 5BE1C29E
 P 1600 7450
@@
 Connection ~ 2000 6950
 $Comp
-L GMcounter-rescue:GND #PWR010
+L GMcounter-rescue:GND-GMcounter-rescue #PWR010
 U 1 1 5BE1C970
 P 9500 850
@@
 	6850 3650 6500 3650
 $Comp
-L GMcounter-rescue:R R10
+L GMcounter-rescue:R-GMcounter-rescue R10
 U 1 1 5BE1D4C8
 P 9850 6100
@@
 $EndComp
 $Comp
-L GMcounter-rescue:R R11
+L GMcounter-rescue:R-GMcounter-rescue R11
 U 1 1 5BE1D5A6
 P 10100 6200
@@
 	10500 6100 10000 6100
 $Comp
-L GMcounter-rescue:+5V #PWR011
+L GMcounter-rescue:+5V-GMcounter-rescue #PWR011
 U 1 1 5BE1DE07
 P 9450 4450
@@
 Connection ~ 9450 4150
 $Comp
-L GMcounter-rescue:USB_A P4
+L GMcounter-rescue:USB_A-GMcounter-rescue P4
 U 1 1 5BE1E114
 P 5050 5000
@@
 $EndComp
 $Comp
-L GMcounter-rescue:+5V #PWR012
+L GMcounter-rescue:+5V-GMcounter-rescue #PWR012
 U 1 1 5BE1E1BC
 P 4400 5450
@@
 D-
 $Comp
-L GMcounter-rescue:GND #PWR013
+L GMcounter-rescue:GND-GMcounter-rescue #PWR013
 U 1 1 5BE1E54E
 P 5450 5450
@@
 Connection ~ 9450 3950
 $Comp
-L GMcounter-rescue:C C8
+L GMcounter-rescue:C-GMcounter-rescue C8
 U 1 1 5BE21F01
 P 9850 4150
@@
 $EndComp
 $Comp
-L GMcounter-rescue:GND #PWR014
+L GMcounter-rescue:GND-GMcounter-rescue #PWR014
 U 1 1 5BE22037
 P 9850 4450
@@
 Connection ~ 9450 3750
 $Comp
-L GMcounter-rescue:R R12
+L GMcounter-rescue:R-GMcounter-rescue R12
 U 1 1 5BE22566
 P 3450 6950
@@
 $EndComp
 $Comp
-L GMcounter-rescue:LED D3
+L GMcounter-rescue:LED-GMcounter-rescue D3
 U 1 1 5BE2261A
 P 3100 6600
@@
 	3450 6600 3300 6600
 $Comp
-L GMcounter-rescue:R R14
+L GMcounter-rescue:R-GMcounter-rescue R14
 U 1 1 5BE23669
 P 9650 2850
@@
 $EndComp
 $Comp
-L GMcounter-rescue:+5V #PWR015
+L GMcounter-rescue:+5V-GMcounter-rescue #PWR015
 U 1 1 5BE236F8
 P 10000 2950
@@
 	10000 2850 10000 2950
 $Comp
-L GMcounter-rescue:CSTLA_T Q4
+L GMcounter-rescue:CSTLA_T-GMcounter-rescue Q4
 U 1 1 5BE238C4
 P 9650 2200
@@
 	9650 1950 9650 2000
 $Comp
-L GMcounter-rescue:GND #PWR016
+L GMcounter-rescue:GND-GMcounter-rescue #PWR016
 U 1 1 5BE23CE5
 P 10150 1900
@@
 	10150 2200 10150 1900
 $Comp
-L GMcounter-rescue:R R13
+L GMcounter-rescue:R-GMcounter-rescue R13
 U 1 1 5BE240ED
 P 6550 1350
@@
 $EndComp
 $Comp
-L GMcounter-rescue:GND #PWR017
+L GMcounter-rescue:GND-GMcounter-rescue #PWR017
 U 1 1 5BE241C1
 P 5650 1350
@@
 $EndComp
 $Comp
-L GMcounter-rescue:LED D4
+L GMcounter-rescue:LED-GMcounter-rescue D4
 U 1 1 5BE2423E
 P 6050 1350
@@
 	6700 1350 6850 1350
 $Comp
-L GMcounter-rescue:C C9
+L GMcounter-rescue:C-GMcounter-rescue C9
 U 1 1 5BE24FD5
 P 10250 2900
@@
 	10250 3250 10250 3050
 $Comp
-L GMcounter-rescue:GND #PWR018
+L GMcounter-rescue:GND-GMcounter-rescue #PWR018
 U 1 1 5BE251E4
 P 10350 2550
@@
 Connection ~ 10250 2550
 $Comp
-L GMcounter-rescue:D D5
+L GMcounter-rescue:D-GMcounter-rescue D5
 U 1 1 5BE258EC
 P 4600 5450
@@
 	4400 5450 4450 5450
 $Comp
-L GMcounter-rescue:CONN_01X03 P5
+L GMcounter-rescue:CONN_01X03-GMcounter-rescue P5
 U 1 1 5BE26104
 P 3500 900
@@
 $EndComp
 $Comp
-L GMcounter-rescue:+5V #PWR019
+L GMcounter-rescue:+5V-GMcounter-rescue #PWR019
 U 1 1 5BE263F9
 P 3700 1200
@@
 	8200 5550 8000 5550
 $Comp
-L GMcounter-rescue:+5V #PWR020
+L GMcounter-rescue:+5V-GMcounter-rescue #PWR020
 U 1 1 5BE27409
 P 8100 5350
@@
 $EndComp
 $Comp
-L GMcounter-rescue:GND #PWR021
+L GMcounter-rescue:GND-GMcounter-rescue #PWR021
 U 1 1 5BE27495
 P 8550 5650
@@
 	6850 2950 6700 2950
 $Comp
-L GMcounter-rescue:+3.3V #PWR022
+L GMcounter-rescue:+3.3V-GMcounter-rescue #PWR022
 U 1 1 5BE29C6A
 P 4900 6700
@@
 $EndComp
 $Comp
-L GMcounter-rescue:CONN_01X03 P7
+L GMcounter-rescue:CONN_01X03-GMcounter-rescue P7
 U 1 1 5BE29C70
 P 5100 6400
@@
 $EndComp
 $Comp
-L GMcounter-rescue:+5V #PWR023
+L GMcounter-rescue:+5V-GMcounter-rescue #PWR023
 U 1 1 5BE29C76
 P 5300 6700
@@
 	5200 6700 5200 6600
 $Comp
-L GMcounter-rescue:GND #PWR024
+L GMcounter-rescue:GND-GMcounter-rescue #PWR024
 U 1 1 5BE29D07
 P 5100 6850
