File: 32u4/GMcounter.kicad_pcb (KiCad board)
At the start: 2 copper layers, 120.4 x 29 mm, 45 parts, among them J1 Conn_02x05_Counter_Clockwise, P1 CONN_01X01, P2 CONN_01X01, P3 CONN_01X01, P4 USB_A, P5 CONN_01X03, P7 CONN_01X03, Q1 MMBT3904, Q2 STL128DN, Q3 MMBT3904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

Commit message: added pic
Other:
- board text added: "Based on MightOhm's Geiger"
Changed lines of the file:
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@@
   (general
     (thickness 1.6)
-    (drawings 9)
+    (drawings 10)
     (tracks 550)
     (zones 0)
@@
       (net 27 "Net-(L1-Pad2)"))
   )
+  (gr_text "Based on MightOhm's\nGeiger" (at 90.932 67.818) (layer B.SilkS)
+    (effects (font (size 1.5 1.5) (thickness 0.3)) (justify mirror))
+  )
   (gr_text "GMCounter 32u4\nTakigama@github" (at 90.932 59.182) (layer B.SilkS)
