File: PINDiode/pindiode/pindiode.kicad_pcb (KiCad board)
At the start: 2 copper layers, 79.8 x 21.3 mm, 34 parts, among them J1 Conn_01x02, J2 Conn_02x05_Counter_Clockwise, J3 Conn_01x02, P1 USB_A, Q1 BF545C, Q2 CSTLA_T, U1 LM358, U2 ATmega32U4-AU

Commit message: per-auto router
Parts:
- moved D2 4.60 mm to (209.8, 75.7), turned to 90 degrees
- moved C9 3.03 mm to (204.8, 80.2)
- moved J1 2.59 mm to (212.3, 68.6)
Routing:
- net GND: track 4.41 -> 37.0 mm, vias 0 -> 11
- net COUNTER: track 24.9 -> 0.00 mm, vias 3 -> 0
- added copper zone on B.Cu, net GND

Commit message: added pic
Parts:
- moved J2 15.5 mm to (179.8, 68.1), turned to 0 degrees
- moved R12 11.8 mm to (173.2, 81.4), turned to 90 degrees
- moved D3 9.48 mm to (176.3, 76.8), turned to 270 degrees
- moved R14 8.90 mm to (176.3, 81.3)
- moved J3 8.46 mm to (179.8, 82.3)
- moved C7 4.69 mm to (173.2, 75.8)
- moved R10 2.99 mm to (173.2, 70.5)
Routing:
- net +5V: track 0.00 -> 64.1 mm
- net MOSI: track 0.00 -> 49.9 mm
- net MISO: track 0.00 -> 49.6 mm
- net RST: track 0.00 -> 42.0 mm
- net COUNTER: track 0.00 -> 33.6 mm
- net SDA: track 0.00 -> 29.4 mm, vias 0 -> 1
- net Net-(Q1-Pad1): track 0.00 -> 27.7 mm
- net Net-(C5-Pad1): track 0.00 -> 25.8 mm
- net SCLK: track 0.00 -> 23.9 mm, vias 0 -> 1
- net Net-(C4-Pad2): track 0.00 -> 23.2 mm
- net SCL: track 0.00 -> 20.1 mm
- net Net-(C7-Pad2): track 0.00 -> 19.8 mm
- net Net-(C4-Pad1): track 0.00 -> 19.2 mm, vias 0 -> 2
- net Net-(R14-Pad1): track 0.00 -> 17.2 mm
- net ADC1: track 0.00 -> 16.4 mm, vias 0 -> 1
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Other:
- board text added: "Based on Elektor's Design"
- board text added: "PINDiode Geiger takigama@github"
